Commit message: feat: Robotiq-style parallel-jaw gripper + pick-and-pour task
URDF (ur5e.urdf):
- Replace fixed gripper_base+beaker with Robotiq 2F-85 inspired gripper
- gripper_body (85x55x40mm) + gripper_coupler + gripper_tip
- left/right_finger with prismatic joints (0-40mm travel)
- left/right_finger_pad (rubber contact surfaces)
- Beaker removed from URDF (now a free object in simulation)

Parser (urdf_parser.py):
- Support prismatic joints in _build_chain() and forward_kinematics()
- Prismatic FK: translation along axis * joint_position

Simulation (pour_task.py):
- Complete rewrite: 5-phase task (APPROACH->GRASP->LIFT->POUR->DONE)
- Source beaker as free object with gravity + bench support
- Gripper grasp detection: proximity + finger closure
- Finger control via action[6]: -1=close, +1=open
- Home pose tool-DOWN [0.4,-0.8,1.2,-1.97,-1.57,pi]
- 56-dim obs, 7-dim action (6 arm vel + 1 grip cmd)
- Phase-specific rewards with dense shaping
- Domain randomization on beaker/glass positions

Dashboard (dashboard.html):
- Prismatic joint handling in updateJoints (translate vs rotate)
- Source beaker as standalone Three.js mesh (tracks telemetry)
- Beaker follows gripper orientation when grasped
- Phase-specific EE glow colors (approach/grasp/lift/pour/done)
- Pour particles emit from beaker position
- Updated SIM defaults for new task phases

Server (server.py):
- Telemetry sends 8 joint values (6 arm + 2 finger)
- New fields: finger_q, gripper_openness, beaker_on_bench

All 26 tests pass.

File: philos/simulation/assets/ur5e.urdf (robot description, URDF)
Before this commit: robot ur5e, 12 links, 11 joints
Links:
- removed link beaker
- removed link gripper_base
- added link gripper_body, mass 0.68; collision box size=0.085 0.055 0.040; visual box size=0.085 0.055 0.040
- added link gripper_coupler, mass 0.08; visual box size=0.070 0.040 0.008
- added link gripper_tip, mass 0.001; visual sphere radius=0.004
- added link left_finger, mass 0.05; collision box size=0.012 0.022 0.060; visual box size=0.012 0.022 0.060
- added link left_finger_pad, mass 0.01; visual box size=0.010 0.020 0.018
- added link right_finger, mass 0.05; collision box size=0.012 0.022 0.060; visual box size=0.012 0.022 0.060
- added link right_finger_pad, mass 0.01; visual box size=0.010 0.020 0.018
Joints:
- removed joint beaker_fixed
- removed joint gripper_fixed
- added joint gripper_body_fixed: type fixed, parent tool0, child gripper_body, origin xyz=0 0 0.005 rpy=0 0 0
- added joint gripper_coupler_fixed: type fixed, parent gripper_body, child gripper_coupler, origin xyz=0 0 0.040 rpy=0 0 0
- added joint gripper_tip_fixed: type fixed, parent gripper_coupler, child gripper_tip, origin xyz=0 0 0.078 rpy=0 0 0
- added joint left_finger_joint: type prismatic, parent gripper_coupler, child left_finger, origin xyz=-0.008 0 0.008 rpy=0 0 0, axis -1 0 0, limit lower=0 upper=0.040 effort=20.0 velocity=0.5
- added joint left_pad_fixed: type fixed, parent left_finger, child left_finger_pad, origin xyz=0 0 0.060 rpy=0 0 0
- added joint right_finger_joint: type prismatic, parent gripper_coupler, child right_finger, origin xyz=0.008 0 0.008 rpy=0 0 0, axis 1 0 0, limit lower=0 upper=0.040 effort=20.0 velocity=0.5
- added joint right_pad_fixed: type fixed, parent right_finger, child right_finger_pad, origin xyz=0 0 0.060 rpy=0 0 0
